Commit message: added arm rotation for picking up trash

File: cerberus_gazebo/models/rover/model.urdf (robot description, URDF)
Before this commit: robot artpark, 15 links, 14 joints
Joints:
- removed joint base_JOINT_1
- added joint robot_manipulator: type revolute, parent base_link, child link_1, axis 0 0 1, limit lower=-3.14 upper=3.14 effort=100 velocity=0.5

Commit message: fixed bot navigation stack

File: cerberus_gazebo/models/rover/model.urdf (robot description, URDF)
Before this commit: robot artpark, 15 links, 14 joints
Joints:
- joint kinect_base: origin xyz=1.70 0.57 0.2 rpy=-1.57 0 -1.57 -> xyz=0.270 0 0.2 rpy=-1.57 0 -1.57
